File: rustypill.kicad_pcb (KiCad board)
At the start: 2 copper layers, 40 parts, among them IC1 DS3231, J1 USB_B_Micro, J2 Conn_01x04, J3 Conn_01x16, J4 Conn_01x16, SW1 Reset, U1 AMS1117-3.3, U2 AT24C512C-SSHD-T, U3 ESP-12F, U4 STM32F103C8Tx, Y1 8MHz

Commit message: ...
Parts:
- added C15: 100nF, Capacitors_SMD:C_0805_HandSoldering, B.Cu at (82.3, 131.7)
- added J5: LCD1602, lib:PinHeader_1x16_P2.54mm_Vertical, F.Cu at (88.3, 97.0)
- added J6: IDC_10P, lib:IDC-Header_2x05_P2.54mm_Vertical, F.Cu at (87.2, 131.2)
- added R13: RCON, Resistors_SMD:R_0805_HandSoldering, B.Cu at (79.0, 102.5)
- added R14: 10k, Resistors_SMD:R_0805_HandSoldering, F.Cu at (73.8, 127.2)
- added REF**: MountingHole_2.7mm_M2.5, Mounting_Holes:MountingHole_2.7mm_M2.5, F.Cu at (133.0, 136.0)
- added REF**: MountingHole_2.7mm_M2.5, Mounting_Holes:MountingHole_2.7mm_M2.5, F.Cu at (72.1, 135.7)
- added REF**: MountingHole_2.7mm_M2.5, Mounting_Holes:MountingHole_2.7mm_M2.5, F.Cu at (133.0, 99.0)
- added REF**: MountingHole_2.7mm_M2.5, Mounting_Holes:MountingHole_2.7mm_M2.5, F.Cu at (72.0, 98.5)
- C1, C10, C11, C12, C13, C14, C2, C3, C6, C7, C8, C9, IC1, R1, R10, R11, R12, R2, R3, R4, R5, R6, R7, R8, U2, U3: moved to B.Cu
- J1: value USB_B_Micro -> USB; moved to B.Cu
- J2: value Conn_01x04 -> PROG
- J3: value Conn_01x16 -> GPIOB
- J4: value Conn_01x16 -> GPIOA
- U4: footprint Housings_QFP:LQFP-48_7x7mm_Pitch0.5mm -> STM32F103C8T6:QFP50P900X900X160-48N
- moved C10 100.4 mm to (73.8, 123.7), turned to 315 degrees
- moved C9 97.7 mm to (75.3, 122.1), turned to 315 degrees
- moved R7 94.1 mm to (77.3, 130.8), turned to 135 degrees
- moved R2 85.5 mm to (74.1, 112.8), turned to 45 degrees
- moved R1 84.6 mm to (85.8, 110.3)
- moved C8 80.6 mm to (85.9, 122.3), turned to 45 degrees
- moved C5 77.8 mm to (92.3, 108.0)
- moved R9 75.3 mm to (72.2, 128.8), turned to 135 degrees
- moved U1 74.9 mm to (90.7, 115.4), turned to 180 degrees
- moved C6 74.5 mm to (77.7, 106.7), turned to 90 degrees
- moved D2 74.0 mm to (85.8, 110.3)
- moved C7 73.2 mm to (84.3, 120.8), turned to 45 degrees
- moved U2 70.5 mm to (102.1, 108.2), turned to 270 degrees
- moved C11 69.5 mm to (100.0, 127.2), turned to 270 degrees
- moved C2 69.4 mm to (90.3, 121.8), turned to 270 degrees
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Connections:
- J4 pad 9: 32KHZ_IN -> A8
- U4 pad 29: 32KHZ_IN -> A8
Other:
- board outline added: 69 x 45.5 mm

Commit message: ...
Parts:
- removed REF** (x3): MountingHole_2.7mm_M2.5, Mounting_Holes:MountingHole_2.7mm_M2.5
- added M2: MountingHole_2.7mm_M2.5, Mounting_Holes:MountingHole_2.7mm_M2.5, F.Cu at (133.0, 99.0)
- added M3: MountingHole_2.7mm_M2.5, Mounting_Holes:MountingHole_2.7mm_M2.5, F.Cu at (72.1, 135.7)
- added M4: MountingHole_2.7mm_M2.5, Mounting_Holes:MountingHole_2.7mm_M2.5, F.Cu at (133.0, 136.0)
-  M1: renamed from REF**
- IC1: moved to F.Cu
- moved R13 45.0 mm to (123.9, 104.6), turned to 180 degrees
- moved J5 38.1 mm to (126.4, 96.9), turned to 270 degrees
- moved IC1 23.6 mm to (124.0, 127.9), turned to 0 degrees
- moved C1 11.7 mm to (103.2, 117.0)
- moved C3 11.7 mm to (100.0, 120.3)
- moved SW1 1.00 mm to (78.5, 107.4)
- moved C6 1.00 mm to (78.5, 107.3)
- moved U1 0.76 mm to (91.5, 115.4)
- moved R8 0.65 mm to (118.5, 104.6)
- moved D1 0.62 mm to (92.2, 110.3)
- moved Y1 0.27 mm to (86.0, 106.6)
- moved D2 0.20 mm to (86.0, 110.3)
- moved R1 0.20 mm to (86.0, 110.3)
- moved C5 0.15 mm to (92.3, 107.8)
Routing:
- net A11: track 0.00 -> 126.2 mm, vias 0 -> 1
- net B14: track 0.00 -> 77.5 mm, vias 0 -> 1
- net B15: track 0.00 -> 51.9 mm, vias 0 -> 1
- net B12: track 0.00 -> 51.2 mm
- net A12: track 0.00 -> 49.2 mm, vias 0 -> 2
- net A8: track 0.00 -> 36.3 mm
- net A9: track 0.00 -> 35.5 mm
- net A10: track 0.00 -> 35.1 mm
- net B13: track 0.00 -> 32.5 mm
- net A13: track 0.00 -> 23.9 mm
- net USB_DP: track 0.00 -> 8.85 mm
- added copper zone on B.Cu, net GND
- added copper zone on F.Cu, net GND

Commit message: ...
Parts:
- removed SW1: Reset, Buttons_Switches_SMD:SW_SPST_SKQG
- moved R6 0.62 mm to (112.5, 104.5)
- moved C7 0.58 mm to (84.0, 121.3)
- moved C8 0.58 mm to (85.6, 122.8)
- moved M2 0.50 mm to (133.0, 98.5)
- moved J2 0.43 mm to (76.7, 96.8)
- moved J4 0.40 mm to (126.7, 100.7)
- moved M3 0.32 mm to (72.0, 136.0)
- moved J5 0.32 mm to (126.7, 96.8)
- moved R8 0.32 mm to (118.2, 104.5)
- moved R13 0.11 mm to (124.0, 104.5)
Routing:
- net +3V3: track 0.00 -> 267.0 mm, vias 0 -> 6
- net B4: track 0.00 -> 155.2 mm, vias 0 -> 1
- net B5: track 0.00 -> 143.8 mm, vias 0 -> 1
- net B3: track 0.00 -> 115.0 mm, vias 0 -> 2
- net B13: track 32.5 -> 122.8 mm, vias 0 -> 1
- net A11: track 126.2 -> 40.5 mm, vias 1 -> 0
- net A0: track 0.00 -> 84.8 mm, vias 0 -> 1
- net B12: track 51.2 -> 129.3 mm, vias 0 -> 2
- net A7: track 0.00 -> 77.0 mm, vias 0 -> 5
- net B0: track 0.00 -> 74.2 mm, vias 0 -> 4
- net B8: track 0.00 -> 73.4 mm, vias 0 -> 2
- net A2: track 0.00 -> 69.1 mm, vias 0 -> 4
- net B1: track 0.00 -> 69.1 mm, vias 0 -> 1
- net A3: track 0.00 -> 67.1 mm, vias 0 -> 5
- net B2: track 0.00 -> 67.0 mm, vias 0 -> 1
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Other:
- outline, holes or cut-outs redrawn

Commit message: ...
Parts:
- moved C8 0.63 mm to (86.1, 123.1)
Routing:
- net B9: track 50.3 -> 158.0 mm, vias 2 -> 9
- net GND: track 65.1 -> 169.2 mm, vias 6 -> 16
- net B8: track 73.4 -> 138.7 mm, vias 2 -> 5
- net B7: track 48.3 -> 105.9 mm, vias 1 -> 4
- net Net-(BT1-Pad1): track 0.00 -> 53.6 mm, vias 0 -> 4
- net 32KHZ_IN: track 0.00 -> 49.3 mm, vias 0 -> 3
- net B6: track 50.2 -> 93.6 mm, vias 1 -> 4
- net +3V3: track 267.0 -> 306.5 mm, vias 6 -> 8
- net A1: track 62.0 -> 99.9 mm, vias 2 -> 3
- net Net-(C4-Pad1): track 10.8 -> 44.8 mm, vias 0 -> 2
- net A2: track 69.1 -> 102.4 mm, vias 4 -> 5
- net VPP: track 52.8 -> 85.3 mm, vias 3 -> 4
- net A4: track 62.0 -> 90.3 mm, vias 2 -> 3
- net A11: track 40.5 -> 65.8 mm, vias 0 -> 1
- net B14: track 110.2 -> 134.1 mm
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
Commit message: ...
Routing:
- net Net-(C5-Pad1): track 5.22 -> 32.8 mm, vias 0 -> 2
- net +3V3: track 306.5 -> 298.4 mm
- net B14: track 134.1 -> 128.9 mm
- net Net-(C7-Pad2): track 17.5 -> 13.1 mm, vias 3 -> 2
- net B12: track 141.0 -> 144.8 mm
- net B15: track 84.2 -> 87.8 mm
- net Net-(D2-Pad1): track 0.00 -> 3.29 mm, vias 0 -> 1
- net Net-(C6-Pad1): track 15.1 -> 18.4 mm
- net A1: track 99.9 -> 97.3 mm
- net B8: track 138.7 -> 136.7 mm
- net GND: track 169.2 -> 170.7 mm, vias 16 -> 13
- net B1: track 71.0 -> 69.7 mm
- net A11: track 65.8 -> 66.7 mm
- net B2: track 69.0 -> 68.0 mm
- net A12: track 58.6 -> 59.4 mm
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- removed copper zone on B.Cu, net GND

Commit message: ...
Routing:
- net B9: track 157.3 -> 100.4 mm, vias 9 -> 6
- net +3V3: track 298.4 -> 331.4 mm, vias 8 -> 9
- net Net-(C6-Pad1): track 18.4 -> 35.1 mm
- net B13: track 121.3 -> 137.8 mm
- net GND: track 170.7 -> 157.2 mm
- net B0: track 89.5 -> 80.3 mm
- net A9: track 81.4 -> 90.1 mm
- net A8: track 41.6 -> 48.3 mm
- net A11: track 66.7 -> 73.1 mm
- net A12: track 59.4 -> 65.3 mm
- net Net-(C5-Pad1): track 32.8 -> 38.1 mm
- net A14: track 45.9 -> 51.0 mm
- net Net-(BT1-Pad1): track 53.6 -> 48.8 mm
- net A13: track 39.4 -> 44.3 mm
- net B8: track 136.7 -> 131.9 mm
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- added copper zone on B.Cu, net GND

Commit message: ...
Routing:
- net +3V3: track 331.4 -> 319.3 mm
Changed lines of the file:
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@@
     (thickness 1.6)
     (drawings 8)
-    (tracks 1914)
+    (tracks 1900)
     (zones 0)
     (modules 48)
@@
   (segment (start 99.294999 137.264001) (end 99.905999 137.875001) (width 0.25) (layer B.Cu) (net 4))
   (segment (start 99.905999 137.875001) (end 101.034001 137.875001) (width 0.25) (layer B.Cu) (net 4))
-  (segment (start 101.034001 137.875001) (end 101.645001 137.264001) (width 0.25) (layer B.Cu) (net 4))
-  (segment (start 101.645001 137.264001) (end 101.645001 136.135999) (width 0.25) (layer B.Cu) (net 4))
-  (segment (start 100.775001 134.751999) (end 100.47501 134.452008) (width 0.25) (layer B.Cu) (net 4))
-  (segment (start 101.645001 136.135999) (end 100.775001 135.265999) (width 0.25) (layer B.Cu) (net 4))
-  (segment (start 100.775001 135.265999) (end 100.775001 134.751999) (width 0.25) (layer B.Cu) (net 4))
-  (segment (start 100.47501 134.452008) (end 100.452008 134.452008) (width 0.25) (layer B.Cu) (net 4))
-  (segment (start 100.452008 134.452008) (end 99.75 133.75) (width 0.25) (layer B.Cu) (net 4))
-  (segment (start 100.75 131.150179) (end 100.373001 130.77318) (width 0.25) (layer B.Cu) (net 4))
-  (segment (start 100.373001 130.77318) (end 99.42682 130.77318) (width 0.25) (layer B.Cu) (net 4))
-  (segment (start 100.75 131.846183) (end 100.75 131.150179) (width 0.25) (layer B.Cu) (net 4))
-  (segment (start 99.75 133.75) (end 99.75 132.846183) (width 0.25) (layer B.Cu) (net 4))
-  (segment (start 99.75 132.846183) (end 100.75 131.846183) (width 0.25) (layer B.Cu) (net 4))
-  (segment (start 99.049999 127.025001) (end 100 126.075) (width 0.25) (layer B.Cu) (net 4))
-  (segment (start 100 126.075) (end 100 125.95) (width 0.25) (layer B.Cu) (net 4))
-  (segment (start 99.049999 130.396359) (end 99.049999 127.025001) (width 0.25) (layer B.Cu) (net 4))
-  (segment (start 99.42682 130.77318) (end 99.049999 130.396359) (width 0.25) (layer B.Cu) (net 4))
   (segment (start 115.05 127.5) (end 115.05 125.3) (width 0.25) (layer B.Cu) (net 4))
   (segment (start 111.7 125.3) (end 111.55 125.15) (width 0.25) (layer B.Cu) (net 4))
@@
   (segment (start 121 126.5) (end 118.785 126.5) (width 0.25) (layer B.Cu) (net 4))
   (segment (start 93.75 120.5) (end 93.75 120.375) (width 0.25) (layer B.Cu) (net 4))
-  (segment (start 101.834999 137.264001) (end 102.445999 137.875001) (width 0.25) (layer B.Cu) (net 4))
-  (segment (start 121.360009 130.899999) (end 120.96001 130.5) (width 0.25) (layer B.Cu) (net 4))
-  (segment (start 124.505001 137.264001) (end 124.505001 134.044991) (width 0.25) (layer B.Cu) (net 4))
   (segment (start 120.86 132.5) (end 120.86 130.60001) (width 0.25) (layer F.Cu) (net 4))
-  (segment (start 99.049999 127.025001) (end 99.049999 129.460001) (width 0.25) (layer B.Cu) (net 4))
   (segment (start 121 126.5) (end 121 130.46001) (width 0.25) (layer F.Cu) (net 4))
   (segment (start 120.86 130.60001) (end 120.96001 130.5) (width 0.25) (layer F.Cu) (net 4))
-  (segment (start 101.834999 136.161409) (end 101.834999 137.264001) (width 0.25) (layer B.Cu) (net 4))
-  (segment (start 123.894001 137.875001) (end 124.505001 137.264001) (width 0.25) (layer B.Cu) (net 4))
   (segment (start 121 130.46001) (end 120.96001 130.5) (width 0.25) (layer F.Cu) (net 4))
-  (segment (start 100.82499 131.234992) (end 100.82499 135.1514) (width 0.25) (layer B.Cu) (net 4))
-  (segment (start 99.049999 129.460001) (end 100.82499 131.234992) (width 0.25) (layer B.Cu) (net 4))
   (via (at 120.96001 130.5) (size 0.8) (drill 0.4) (layers F.Cu B.Cu) (net 4))
-  (segment (start 100.82499 135.1514) (end 101.834999 136.161409) (width 0.25) (layer B.Cu) (net 4))
-  (segment (start 102.445999 137.875001) (end 123.894001 137.875001) (width 0.25) (layer B.Cu) (net 4))
-  (segment (start 124.505001 134.044991) (end 121.360009 130.899999) (width 0.25) (layer B.Cu) (net 4))
   (segment (start 94.3 125.9) (end 94.4 125.9) (width 0.25) (layer B.Cu) (net 4))
   (segment (start 97.2 123.1) (end 97.2 122.623002) (width 0.25) (layer B.Cu) (net 4))
@@
   (segment (start 89.699998 108.2) (end 86.149998 104.65) (width 0.25) (layer B.Cu) (net 4))
   (segment (start 86.149998 104.65) (end 79.2 104.65) (width 0.25) (layer B.Cu) (net 4))
+  (segment (start 120.96001 130.5) (end 124.505001 134.044991) (width 0.25) (layer B.Cu) (net 4))
+  (segment (start 124.505001 137.264001) (end 123.894001 137.875001) (width 0.25) (layer B.Cu) (net 4))
+  (segment (start 124.505001 134.044991) (end 124.505001 137.264001) (width 0.25) (layer B.Cu) (net 4))
+  (segment (start 123.894001 137.875001) (end 102.445999 137.875001) (width 0.25) (layer B.Cu) (net 4))
+  (segment (start 101.034001 137.875001) (end 102.445999 137.875001) (width 0.25) (layer B.Cu) (net 4))
+  (segment (start 99.049999 127.025001) (end 100 126.075) (width 0.25) (layer B.Cu) (net 4))
+  (segment (start 99.049999 129.460001) (end 99.049999 127.025001) (width 0.25) (layer B.Cu) (net 4))
+  (segment (start 101.834999 137.264001) (end 101.834999 132.235178) (width 0.25) (layer B.Cu) (net 4))
+  (segment (start 102.445999 137.875001) (end 101.834999 137.264001) (width 0.25) (layer B.Cu) (net 4))
+  (segment (start 101.834999 132.235178) (end 100.373001 130.77318) (width 0.25) (layer B.Cu) (net 4))
+  (segment (start 100.373001 130.77318) (end 100.363178 130.77318) (width 0.25) (layer B.Cu) (net 4))
+  (segment (start 100 126.075) (end 100 125.95) (width 0.25) (layer B.Cu) (net 4))
+  (segment (start 100.363178 130.77318) (end 99.049999 129.460001) (width 0.25) (layer B.Cu) (net 4))
   (segment (start 91.05 104.45) (end 91.05 105.325) (width 0.25) (layer F.Cu) (net 5))
   (segment (start 90.599986 103.999986) (end 91.05 104.45) (width 0.25) (layer F.Cu) (net 5))

Commit message: ...
Parts:
- added SW1: Reset, Buttons_Switches_SMD:SW_SPST_SKQG, F.Cu at (125.7, 111.5)
- moved C11 18.5 mm to (118.2, 130.8)
- moved  M1 2.50 mm to (72.0, 96.0)
- moved M2 2.50 mm to (133.0, 96.0)
- moved J3 1.66 mm to (127.3, 135.9)
- moved C8 1.07 mm to (86.8, 122.3)
- moved C15 1.07 mm to (83.0, 130.9)
- moved C10 1.07 mm to (74.4, 122.8)
- moved C13 1.07 mm to (112.2, 125.5)
- moved C4 1.07 mm to (93.0, 104.5)
- moved IC1 1.07 mm to (124.7, 127.0)
- moved R10 1.07 mm to (78.0, 124.5)
- moved R11 1.07 mm to (79.7, 126.3)
- moved R14 1.07 mm to (74.5, 126.3)
- moved J4 1.07 mm to (127.3, 99.8)
- moved R12 1.07 mm to (96.3, 125.0)
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Routing:
- net GND: track 157.2 -> 349.5 mm, vias 13 -> 10
- net Net-(C6-Pad1): track 35.1 -> 137.3 mm, vias 1 -> 2
- net +3V3: track 319.3 -> 220.9 mm, vias 9 -> 11
- net B12: track 147.7 -> 103.4 mm
- net A2: track 101.0 -> 134.1 mm, vias 5 -> 1
- net B8: track 131.9 -> 101.4 mm, vias 5 -> 7
- net B11: track 39.1 -> 68.3 mm, vias 1 -> 4
- net A9: track 90.1 -> 62.6 mm, vias 5 -> 2
- net Net-(BT1-Pad1): track 48.8 -> 21.9 mm, vias 4 -> 2
- net B10: track 63.5 -> 38.0 mm, vias 1 -> 3
- net B14: track 133.1 -> 111.9 mm, vias 1 -> 2
- net B13: track 137.8 -> 158.7 mm, vias 1 -> 2
- net Net-(C4-Pad1): track 45.7 -> 26.4 mm
- net B0: track 80.3 -> 61.4 mm, vias 4 -> 2
- net B15: track 91.5 -> 73.6 mm
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- removed copper zone on B.Cu, net GND
- removed copper zone on F.Cu, net GND
Other:
- board size 69 x 45.5 mm -> 69 x 48 mm
