File: rustypill.kicad_pcb (KiCad board)
At the start: 2 copper layers, 72 x 52 mm, 56 parts, among them IC1 DS3231, J1 USB, J2 PROG, J3 GPIOB, J4 GPIOA, J5 LCD1602, J6 IDC_10P, J7 I2C, J8 Micro_SD_Card, M2 MountingHole_2.7mm_M2.5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

Commit message: finish routing
Parts:
- Q1: value BC548 -> S8050
- moved J8 1.02 mm to (128.6, 130.0)
Routing:
- net B10: track 132.7 -> 49.5 mm, vias 2 -> 1
- net Net-(C4-Pad1): track 114.1 -> 36.3 mm, vias 12 -> 2
- net A0: track 130.0 -> 73.1 mm, vias 6 -> 0
- net A10: track 112.3 -> 66.7 mm, vias 8 -> 4
- net A11: track 93.3 -> 53.1 mm
- net A7: track 85.5 -> 61.5 mm, vias 3 -> 1
- net B11: track 77.8 -> 56.9 mm, vias 7 -> 1
- net B2: track 95.4 -> 115.1 mm, vias 5 -> 1
- net A12: track 65.7 -> 84.7 mm, vias 3 -> 1
- net B6: track 100.1 -> 82.2 mm, vias 5 -> 1
- net A4: track 87.8 -> 72.2 mm, vias 3 -> 2
- net A6: track 81.2 -> 66.6 mm, vias 2 -> 1
- net Net-(BT1-Pad1): track 75.6 -> 61.2 mm, vias 6 -> 2
- net 32KHZ_IN: track 107.5 -> 94.0 mm, vias 7 -> 1
- net Net-(C1-Pad1): track 37.5 -> 24.2 mm, vias 3 -> 1
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
Commit message: finish routing
Parts:
- removed IC1: DS3231, DS3231:SO16W
- added C18: 4.7uF, Capacitors_SMD:C_0805_HandSoldering, B.Cu at (83.8, 111.5)
- added U6: DS3231, DS3231:SO16W, F.Cu at (113.6, 131.3)
- C14, C2: footprint Capacitors_SMD:C_0805_HandSoldering -> Capacitors_Tantalum_SMD:CP_Tantalum_Case-A_EIA-3216-18_Reflow
- J5: value LCD1602 -> HD44780
- U2: moved to B.Cu
- U4: value STM32F103C8Tx -> STM32F411CEUx; footprint STM32F103C8T6:QFP50P900X900X160-48N -> stm32f411ceu6:QFN50P700X700X60-49N-D
- moved U2 23.5 mm to (100.4, 107.1), turned to 90 degrees
- moved C12 22.7 mm to (104.2, 107.0), turned to 270 degrees
- moved Q1 6.36 mm to (70.8, 108.5), turned to 225 degrees
- moved  M1 2.00 mm to (70.5, 95.7)
- moved M3 2.00 mm to (70.5, 140.3)
- moved U4 0.09 mm to (79.8, 116.2)
Connections:
- Q1 pad 1: LCD_EN -> LCD_BL
- R4 pad 2: B7 -> B6
- R5 pad 2: B6 -> B5
- U3 pad 1: B7 -> B6
- U3 pad 3: B6 -> B5
- U5 pad 7: LCD_BL -> LCD_EN
Routing:
- net A10: track 66.7 -> 138.5 mm, vias 4 -> 3
- net +3V3: track 256.9 -> 311.1 mm, vias 10 -> 6
- net B7: track 100.4 -> 48.3 mm
- net B2: track 115.1 -> 64.1 mm, vias 1 -> 3
- net A9: track 63.6 -> 114.2 mm, vias 1 -> 3
- net Net-(BT1-Pad1): track 61.2 -> 16.9 mm, vias 2 -> 0
- net IC_RST: track 125.8 -> 87.6 mm, vias 8 -> 3
- net B0: track 112.2 -> 75.0 mm, vias 1 -> 2
- net A11: track 53.1 -> 78.9 mm, vias 2 -> 3
- net GND: track 420.6 -> 407.4 mm, vias 7 -> 4
- net A15: track 25.7 -> 38.8 mm, vias 1 -> 3
- net B13: track 107.1 -> 94.6 mm, vias 0 -> 1
- net LCD_RS: track 65.5 -> 53.2 mm, vias 0 -> 2
- net A2: track 59.0 -> 70.0 mm
- net B8: track 144.0 -> 133.5 mm, vias 3 -> 5
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Other:
- board size 72 x 52 mm -> 70 x 52 mm

Commit message: clean up
Parts:
- J2: footprint lib:PinHeader_1x04_P2.54mm_Horizontal -> Pin_Headers:Pin_Header_Angled_1x04_Pitch2.54mm
- J3, J4, J5: footprint lib:PinHeader_1x16_P2.54mm_Vertical -> Pin_Headers:Pin_Header_Straight_1x16_Pitch2.54mm
- J7: footprint lib:PinHeader_1x04_P2.54mm_Vertical -> Pin_Headers:Pin_Header_Straight_1x04_Pitch2.54mm
- U2: footprint AT24C512C-SSHD-T:SOIC127P600X175-8N -> lib:at24c512c-sshd-t
- U4: footprint stm32f411ceu6:QFN50P700X700X60-49N-D -> lib:stm32f411ceu6
- U6: footprint DS3231:SO16W -> lib:ds3231

Commit message: ...
Parts:
- J5, J7: moved to B.Cu
- turned J5 to 90 degrees
- turned J7 to 270 degrees
Routing:
- net B10: track 53.9 -> 54.9 mm
- net IC_RST: track 87.6 -> 88.4 mm

Commit message: ...
Parts:
- added D3: LED, LEDs:LED_0805_HandSoldering, B.Cu at (81.3, 127.9)
- added R16: RLED, Resistors_SMD:R_0805_HandSoldering, B.Cu at (84.0, 124.4)
- added R17: 47k, Resistors_SMD:R_0805_HandSoldering, F.Cu at (119.5, 132.7)
- moved U6 0.66 mm to (113.0, 131.3)
Connections:
- net IC_RST renamed ESP_BOOT0
Routing:
- net Net-(R16-Pad1): track 0.00 -> 4.79 mm, vias 0 -> 1
- net +3V3: track 311.1 -> 315.3 mm
- net Net-(D3-Pad1): track 0.00 -> 3.36 mm
- net GND: track 407.6 -> 410.6 mm
- net B1: track 119.3 -> 121.8 mm
- net B2: track 63.8 -> 65.5 mm
- net 32KHZ_IN: track 101.5 -> 100.4 mm
- net Net-(BT1-Pad1): track 16.9 -> 17.6 mm
- net LCD_RS: track 53.2 -> 53.8 mm

Commit message: finish v0.2.0
Parts:
- moved C11 40.1 mm to (111.7, 130.8), turned to 180 degrees
Routing:
- net A9: track 114.2 -> 121.6 mm, vias 3 -> 1
- net B8: track 133.8 -> 141.1 mm
- net B9: track 140.6 -> 137.8 mm, vias 5 -> 6
- net B1: track 121.8 -> 119.4 mm
- net A11: track 78.9 -> 81.3 mm
- net GND: track 410.6 -> 412.9 mm
- net A10: track 138.5 -> 140.6 mm
- net +3V3: track 315.3 -> 313.3 mm
- net ESP_BOOT0: track 88.7 -> 87.1 mm
- net B2: track 65.5 -> 67.1 mm
- net A12: track 75.0 -> 73.5 mm
- net B15: track 85.9 -> 84.4 mm
- net A0: track 69.8 -> 71.2 mm
- net LCD_EN: track 44.9 -> 46.2 mm
- net B12: track 90.7 -> 89.4 mm
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- added copper zone on B.Cu, net GND
- added copper zone on F.Cu, net GND

Commit message: fix the sdcard orientation issue
Parts:
- moved R17 0.33 mm to (119.5, 133.0)
- moved J8 0.32 mm to (128.6, 129.7), turned to 270 degrees
Routing:
- net B15: track 84.4 -> 100.7 mm
- net GND: track 412.9 -> 428.4 mm, vias 4 -> 5
- net +3V3: track 313.3 -> 326.1 mm
- net B0: track 74.9 -> 87.6 mm
- net B12: track 89.4 -> 95.6 mm
- net B14: track 98.8 -> 93.2 mm
- net B13: track 94.2 -> 93.6 mm
Other:
- board text added: "Rustypill v0.2.1 by Ted"
- board text removed: "Rustypill v0.2.0 by Ted"
