File: rustypill.sch (KiCad schematic (older format))
At the start: 46 parts, among them IC1 DS3231, J1 USB, J2 PROG, J3 GPIOB, J4 GPIOA, J5 LCD1602, J6 IDC_10P, J7 I2C, SW1 Reset, U1 AMS1117-3.3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

Commit message: ...
Parts:
- added C16, C17: 100nF, Capacitors_SMD:C_0805_HandSoldering, symbol Device:C
- added J8: Micro_SD_Card, lib:473340001, symbol Connector:Micro_SD_Card
- added Q1: BC548, TO_SOT_Packages_SMD:SOT-23, symbol Transistor_BJT:BC548
- added R15: Rbl, Resistors_SMD:R_0805_HandSoldering, symbol Device:R_Small
- added U5: PCF8574, lib:VQFN-16-1EP_3x3mm_P0.5mm_EP1.68x1.68mm, symbol Interface_Expansion:PCF8574
Connections:
- net +3V3: now also C16.2, C17.1, J8.4 (VDD), U5.16 (VDD)
- net A15: no longer J5.14 (Pin_14)
- net B12: now also J8.2 (DAT3/CD); no longer J5.4 (Pin_4)
- net B13: now also J8.5 (CLK); no longer J5.5 (Pin_5)
- net B14: now also J8.7 (DAT0); no longer J5.6 (Pin_6)
- net B15: now also J8.3 (CMD); no longer J5.16 (Pin_16)
- net B3: no longer J5.11 (Pin_11)
- net B4: no longer J5.12 (Pin_12)
- net B5: no longer J5.13 (Pin_13)
- net B8: now also U5.14 (SCL)
- net B9: now also U5.15 (SDA)
- net GND: now also C16.1, C17.2, J8.6 (VSS), J8.9 (SHIELD), Q1.3 (E), U5.1 (A0), U5.2 (A1), U5.3 (A2), U5.8 (VSS)
- new net: R15.1, U5.6 (P2)
- new net: Q1.2 (B), R15.2
- new net LCD_BL: J5.16 (Pin_16), U5.7 (P3)
- new net LCD_D4: J5.11 (Pin_11), U5.9 (P4)
- new net LCD_D5: J5.12 (Pin_12), U5.10 (P5)
- new net LCD_D6: J5.13 (Pin_13), U5.11 (P6)
- new net LCD_D7: J5.14 (Pin_14), U5.12 (P7)
- new net LCD_EN: J5.6 (Pin_6), Q1.1 (C)
- new net LCD_RS: J5.4 (Pin_4), U5.4 (P0)
- new net LCD_RW: J5.5 (Pin_5), U5.5 (P1)
- no-connect marks 21 -> 24
Changed lines of the file:
@@
 NoConn ~ 6950 5800
 NoConn ~ 7050 5800
-Text GLabel 7800 4550 0    50   Input ~ 0
+Text GLabel 2550 1300 2    50   Input ~ 0
 LCD_RS
-Wire Wire Line
-	7800 4550 8150 4550
-Text GLabel 7800 4650 0    50   Input ~ 0
+Text GLabel 2550 1400 2    50   Input ~ 0
 LCD_RW
-Wire Wire Line
-	7800 4650 8150 4650
-Text GLabel 7800 4750 0    50   Input ~ 0
-LCD_EN
-Wire Wire Line
-	7800 4750 8150 4750
-Text GLabel 7800 4850 0    50   Input ~ 0
+Text GLabel 2550 1600 2    50   Input ~ 0
 LCD_BL
-Wire Wire Line
-	7800 4850 8150 4850
 $Comp
 L power:+3.3V #PWR0108
@@
 	1    0    0    -1
 $EndComp
-Text GLabel 9800 4850 2    50   Input ~ 0
-LCD_D7
-Wire Wire Line
-	9450 4850 9800 4850
-Text GLabel 7800 3650 0    50   Input ~ 0
+Text GLabel 2550 1700 2    50   Input ~ 0
 LCD_D4
-Text GLabel 7800 3750 0    50   Input ~ 0
+Text GLabel 2550 1800 2    50   Input ~ 0
 LCD_D5
-Text GLabel 7800 3850 0    50   Input ~ 0
+Text GLabel 2550 1900 2    50   Input ~ 0
 LCD_D6
 Connection ~ 7050 3650
@@
 Wire Wire Line
 	7800 3950 8150 3950
-Wire Wire Line
-	7800 3850 8150 3850
-Wire Wire Line
-	7800 3750 8150 3750
-Wire Wire Line
-	7800 3650 8150 3650
 Text GLabel 3500 5600 2    50   Input ~ 0
 A0
@@
 	0    1    1    0
 $EndComp
+$Comp
+L Interface_Expansion:PCF8574 U5
+U 1 1 5DF9CEEE
+P 2050 1700
+F 0 "U5" H 2050 2581 50  0000 C CNN
+F 1 "PCF8574" H 2050 2490 50  0000 C CNN
+F 2 "lib:VQFN-16-1EP_3x3mm_P0.5mm_EP1.68x1.68mm" H 2050 1700 50  0001 C CNN
+F 3 "http://www.nxp.com/documents/data_sheet/PCF8574_PCF8574A.pdf" H 2050 1700 50  0001 C CNN
+	1    2050 1700
+	1    0    0    -1
+$EndComp
+Wire Wire Line
+	8100 3650 8150 3650
+Wire Wire Line
+	8100 3750 8150 3750
+Wire Wire Line
+	8100 3850 8150 3850
+Wire Wire Line
+	9450 4850 9500 4850
+Text GLabel 2550 2000 2    50   Input ~ 0
+LCD_D7
+$Comp
+L power:+3.3V #PWR0111
+U 1 1 5E0D450B
+P 2050 1000
+F 0 "#PWR0111" H 2050 850 50  0001 C CNN
+F 1 "+3.3V" H 2065 1173 50  0000 C CNN
+F 2 "" H 2050 1000 50  0001 C CNN
+F 3 "" H 2050 1000 50  0001 C CNN
+	1    2050 1000
+	1    0    0    -1
+$EndComp
+$Comp
+L power:GND #PWR0112
+U 1 1 5E0D855A
+P 2050 2600
+F 0 "#PWR0112" H 2050 2350 50  0001 C CNN
+F 1 "GND" H 2055 2427 50  0000 C CNN
+F 2 "" H 2050 2600 50  0001 C CNN
+F 3 "" H 2050 2600 50  0001 C CNN
+	1    2050 2600
+	1    0    0    -1
+$EndComp
+Wire Wire Line
+	2050 2600 2050 2550
+$Comp
+L Device:C C16
+U 1 1 5E0E8CA1
+P 1650 2550
+F 0 "C16" H 1765 2596 50  0000 L CNN
+F 1 "100nF" H 1765 2505 50  0000 L CNN
+F 2 "Capacitors_SMD:C_0805_HandSoldering" H 1688 2400 50  0001 C CNN
+F 3 "~" H 1650 2550 50  0001 C CNN
+	1    1650 2550
+	0    1    1    0
+$EndComp
+Wire Wire Line
+	2050 2550 1800 2550
+Connection ~ 2050 2550
+$Comp
+L power:+3.3V #PWR0113
+U 1 1 5E0F8D0C
+P 1400 2550
+F 0 "#PWR0113" H 1400 2400 50  0001 C CNN
+F 1 "+3.3V" H 1415 2723 50  0000 C CNN
+F 2 "" H 1400 2550 50  0001 C CNN
+F 3 "" H 1400 2550 50  0001 C CNN
+	1    1400 2550
+	0    -1   -1   0
+$EndComp
+Wire Wire Line
+	1400 2550 1500 2550
+Wire Wire Line
+	2050 2400 2050 2550
+Wire Wire Line
+	1550 1600 1450 1600
+Wire Wire Line
+	1450 1600 1450 1700
+Wire Wire Line
+	1450 2400 2050 2400
+Connection ~ 2050 2400
+Wire Wire Line
+	1550 1700 1450 1700
+Connection ~ 1450 1700
+Wire Wire Line
+	1450 1700 1450 1800
+Wire Wire Line
+	1550 1800 1450 1800
+Connection ~ 1450 1800
+Wire Wire Line
+	1450 1800 1450 2400
+Text GLabel 1450 1400 0    50   Input ~ 0
+I2C1_SDA
+Wire Wire Line
+	1450 1400 1550 1400
+Text GLabel 1450 1300 0    50   Input ~ 0
+I2C1_SCL
+Wire Wire Line
+	1450 1300 1550 1300
+NoConn ~ 1550 2100
+$Comp
+L Transistor_BJT:BC548 Q1
+U 1 1 5E204241
+P 3300 1500
+F 0 "Q1" H 3491 1546 50  0000 L CNN
+F 1 "BC548" H 3491 1455 50  0000 L CNN
+F 2 "TO_SOT_Packages_SMD:SOT-23" H 3500 1425 50  0001 L CIN
+F 3 "http://www.fairchildsemi.com/ds/BC/BC547.pdf" H 3300 1500 50  0001 L CNN
+	1    3300 1500
+	1    0    0    -1
+$EndComp
+Wire Wire Line
+	3400 1250 3400 1300
+$Comp
+L power:GND #PWR0114
+U 1 1 5E27024D
+P 3400 1800
+F 0 "#PWR0114" H 3400 1550 50  0001 C CNN
+F 1 "GND" H 3405 1627 50  0000 C CNN
+F 2 "" H 3400 1800 50  0001 C CNN
+F 3 "" H 3400 1800 50  0001 C CNN
+	1    3400 1800
+	1    0    0    -1
+$EndComp
+Wire Wire Line
+	3400 1800 3400 1700
+Text GLabel 9150 5850 0    50   Input ~ 0
+SPI_NSS
+Text GLabel 9150 5950 0    50   Input ~ 0
+SPI_MOSI
+Text GLabel 9150 6150 0    50   Input ~ 0
+SPI_SCK
+Text GLabel 9150 6350 0    50   Input ~ 0
+SPI_MISO
+$Comp
+L power:+3.3V #PWR0115
+U 1 1 5E2F046B
+P 8300 5950
+F 0 "#PWR0115" H 8300 5800 50  0001 C CNN
+F 1 "+3.3V" V 8300 6050 50  0000 L CNN
+F 2 "" H 8300 5950 50  0001 C CNN
+F 3 "" H 8300 5950 50  0001 C CNN
+	1    8300 5950
+	1    0    0    -1
+$EndComp
+$Comp
+L power:GND #PWR0116
+U 1 1 5E2F1C11
+P 8300 6350
+F 0 "#PWR0116" H 8300 6100 50  0001 C CNN
+F 1 "GND" H 8200 6200 50  0000 C CNN
+F 2 "" H 8300 6350 50  0001 C CNN
+F 3 "" H 8300 6350 50  0001 C CNN
+	1    8300 6350
+	1    0    0    -1
+$EndComp
+NoConn ~ 9150 5750
+NoConn ~ 9150 6450
+Text GLabel 7800 4550 0    50   Input ~ 0
+SPI_NSS
+Text GLabel 7800 4650 0    50   Input ~ 0
+SPI_SCK
+Text GLabel 7800 4750 0    50   Input ~ 0
+SPI_MISO
+Text GLabel 7800 4850 0    50   Input ~ 0
+SPI_MOSI
+Wire Wire Line
+	7800 4550 8150 4550
+Wire Wire Line
+	7800 4650 8150 4650
+Wire Wire Line
+	7800 4750 8150 4750
+Wire Wire Line
+	7800 4850 8150 4850
+$Comp
+L Device:R_Small R15
+U 1 1 5E381D09
+P 2850 1500
+F 0 "R15" V 2800 1350 50  0000 C CNN
+F 1 "Rbl" V 2900 1350 50  0000 C CNN
+F 2 "Resistors_SMD:R_0805_HandSoldering" H 2850 1500 50  0001 C CNN
+F 3 "~" H 2850 1500 50  0001 C CNN
+	1    2850 1500
+	0    -1   -1   0
+$EndComp
+Wire Wire Line
+	2550 1500 2750 1500
+Wire Wire Line
+	2950 1500 3100 1500
+Wire Wire Line
+	3550 1250 3400 1250
+Text GLabel 3550 1250 2    50   Input ~ 0
+LCD_EN
+$Comp
+L power:GND #PWR0117
+U 1 1 5E3D198F
+P 10850 6650
+F 0 "#PWR0117" H 10850 6400 50  0001 C CNN
+F 1 "GND" H 10750 6500 50  0000 C CNN
+F 2 "" H 10850 6650 50  0001 C CNN
+F 3 "" H 10850 6650 50  0001 C CNN
+	1    10850 6650
+	0    -1   -1   0
+$EndComp
+$Comp
+L Device:C C17
+U 1 1 5E3DAB90
+P 8300 6150
+F 0 "C17" H 8350 6250 50  0000 L CNN
+F 1 "100nF" H 8350 6050 50  0000 L CNN
+F 2 "Capacitors_SMD:C_0805_HandSoldering" H 8338 6000 50  0001 C CNN
+F 3 "~" H 8300 6150 50  0001 C CNN
+	1    8300 6150
+	1    0    0    -1
+$EndComp
+Wire Wire Line
+	8300 6300 8300 6350
+Wire Wire Line
+	8300 6000 8300 5950
+$Comp
+L Connector:Micro_SD_Card J8
+U 1 1 5E29D2F8
+P 10050 6050
+F 0 "J8" H 10000 6767 50  0000 C CNN
+F 1 "Micro_SD_Card" H 10000 6676 50  0000 C CNN
+F 2 "lib:473340001" H 11200 6350 50  0001 C CNN
+F 3 "http://katalog.we-online.de/em/datasheet/693072010801.pdf" H 10050 6050 50  0001 C CNN
+	1    10050 6050
+	1    0    0    -1
+$EndComp
+Wire Wire Line
+	9150 6250 8600 6250
+Wire Wire Line
+	8600 6250 8600 6350
+Wire Wire Line
+	8600 6350 8300 6350
+Connection ~ 8300 6350
+Wire Wire Line
+	9150 6050 8600 6050
+Wire Wire Line
+	8600 6050 8600 5950
+Wire Wire Line
+	8600 5950 8300 5950
+Connection ~ 8300 5950
 $EndSCHEMATC

Commit message: finish routing
Parts:
- Q1: value BC548 -> S8050
Changed lines of the file:
@@
 U 1 1 5E204241
 P 3300 1500
-F 0 "Q1" H 3491 1546 50  0000 L CNN
-F 1 "BC548" H 3491 1455 50  0000 L CNN
+F 0 "Q1" H 3490 1546 50  0000 L CNN
+F 1 "S8050" H 3490 1455 50  0000 L CNN
 F 2 "TO_SOT_Packages_SMD:SOT-23" H 3500 1425 50  0001 L CIN
 F 3 "http://www.fairchildsemi.com/ds/BC/BC547.pdf" H 3300 1500 50  0001 L CNN

Commit message: finish routing
Parts:
- removed U4: STM32F103C8Tx, STM32F103C8T6:QFP50P900X900X160-48N, symbol MCU_ST_STM32F1:STM32F103C8Tx
- added C18: 4.7uF, Capacitors_SMD:C_0805_HandSoldering, symbol Device:C_Small
- added U4: STM32F411CEUx, stm32f411ceu6:QFN50P700X700X60-49N-D, symbol MCU_ST_STM32F4:STM32F411CEUx
- C14, C2: footprint Capacitors_SMD:C_0805_HandSoldering -> Capacitors_Tantalum_SMD:CP_Tantalum_Case-A_EIA-3216-18_Reflow
- J5: value LCD1602 -> HD44780
- renumbered IC1 to U6
Connections:
- net +3V3: now also U4.1 (VBAT), U4.24 (VDD), U4.36 (VDD), U4.48 (VDD)
- net 32KHZ_IN: now also U4.29 (PA8)
- net A0: now also U4.10 (PA0)
- net A1: now also U4.11 (PA1)
- net A10: now also U4.31 (PA10)
- net A11: now also U4.32 (PA11)
- net A12: now also U4.33 (PA12)
- net A13: now also U4.34 (PA13)
- net A14: now also U4.37 (PA14)
- net A15: now also U4.38 (PA15)
- net A2: now also U4.12 (PA2)
- net A3: now also U4.13 (PA3)
- net A4: now also U4.14 (PA4)
- net A5: now also U4.15 (PA5)
- net A6: now also U4.16 (PA6)
- net A7: now also U4.17 (PA7)
- net A9: now also U4.30 (PA9)
- net B0: now also U4.18 (PB0)
- net B1: now also U4.19 (PB1)
- net B10: now also U4.21 (PB10)
- net B11: now also C18.2, U4.22 (VCAP1)
- net B12: now also U4.25 (PB12)
- net B13: now also U4.26 (PB13)
- net B14: now also U4.27 (PB14)
- net B15: now also U4.28 (PB15)
- net B2: now also U4.20 (PB2)
- net B3: now also U4.39 (PB3)
- net B4: now also U4.40 (PB4)
- net B5: now also R5.2, U3.3 (EN), U4.41 (PB5)
- net B6: now also R4.2, U3.1 (~RST), U4.42 (PB6); no longer R5.2, U3.3 (EN)
- net B7: now also U4.43 (PB7); no longer R4.2, U3.1 (~RST)
- net B8: now also U4.45 (PB8)
- net B9: now also U4.46 (PB9)
- net GND: now also C18.1, U4.23 (VSS), U4.35 (VSS), U4.44 (BOOT0), U4.47 (VSS), U4.49 (VSS), U4.8 (VSSA)
- net IC_RST: now also U4.7 (NRST)
- net LCD_BL: now also Q1.1 (C); no longer U5.7 (P3)
- net LCD_EN: now also U5.7 (P3); no longer Q1.1 (C)
- net at C5.1, Y1.2: now also U4.5 (PH0)
- net at C4.1, Y1.1: now also U4.6 (PH1)
- net at C7.2, C8.2, R3.2: now also U4.9 (VDDA)
Other:
- note added: "0.2.0"
- note added: "Rustypill IoT board"
- moved on the sheet: C10, C15, C17, C4, C5, C6, C9, J1, J8, R10, R11, R2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

Commit message: clean up
Parts:
- J2: footprint lib:PinHeader_1x04_P2.54mm_Horizontal -> Pin_Headers:Pin_Header_Angled_1x04_Pitch2.54mm
- J3, J4, J5: footprint lib:PinHeader_1x16_P2.54mm_Vertical -> Pin_Headers:Pin_Header_Straight_1x16_Pitch2.54mm
- J7: footprint lib:PinHeader_1x04_P2.54mm_Vertical -> Pin_Headers:Pin_Header_Straight_1x04_Pitch2.54mm
- U2: footprint AT24C512C-SSHD-T:SOIC127P600X175-8N -> lib:at24c512c-sshd-t
- U4: footprint stm32f411ceu6:QFN50P700X700X60-49N-D -> lib:stm32f411ceu6
- U6: footprint DS3231:SO16W -> lib:ds3231
Changed lines of the file:
@@
 F 0 "U6" H 4750 4626 50  0000 C CNN
 F 1 "DS3231" H 4750 4050 50  0001 L BNN
-F 2 "DS3231:SO16W" H 4750 4050 50  0001 L BNN
+F 2 "lib:ds3231" H 4750 4050 50  0001 L BNN
 F 3 "" H 4750 4050 50  0001 L BNN
 F 4 "Maxim Integrated" H 4750 4050 50  0001 L BNN "Field4"
@@
 F 0 "U2" H 2200 4620 50  0000 C CNN
 F 1 "AT24C512C-SSHD-T" H 2200 4529 50  0000 C CNN
-F 2 "AT24C512C-SSHD-T:SOIC127P600X175-8N" H 2200 3950 50  0001 L BNN
+F 2 "lib:at24c512c-sshd-t" H 2200 3950 50  0001 L BNN
 F 3 "AT24C512C Series 512 Kb _64 K x 8_ 1.7 V I2C-Compatible Serial EEPROM - SOIC-8" H 2200 3950 50  0001 L BNN
 F 4 "Microchip" H 2200 3950 50  0001 L BNN "Field4"
@@
 F 0 "J2" H 2280 5242 50  0000 L CNN
 F 1 "PROG" H 2280 5151 50  0000 L CNN
-F 2 "lib:PinHeader_1x04_P2.54mm_Horizontal" H 2200 5250 50  0001 C CNN
+F 2 "Pin_Headers:Pin_Header_Angled_1x04_Pitch2.54mm" H 2200 5250 50  0001 C CNN
 F 3 "~" H 2200 5250 50  0001 C CNN
 	1    2200 5250
@@
 F 0 "J3" V 5050 6100 50  0000 C CNN
 F 1 "GPIOB" V 5050 5900 50  0000 C CNN
-F 2 "lib:PinHeader_1x16_P2.54mm_Vertical" H 4950 6000 50  0001 C CNN
+F 2 "Pin_Headers:Pin_Header_Straight_1x16_Pitch2.54mm" H 4950 6000 50  0001 C CNN
 F 3 "~" H 4950 6000 50  0001 C CNN
 	1    4950 6000
@@
 F 0 "J4" V 5150 5300 50  0000 C CNN
 F 1 "GPIOA" V 5150 5500 50  0000 C CNN
-F 2 "lib:PinHeader_1x16_P2.54mm_Vertical" H 5050 5500 50  0001 C CNN
+F 2 "Pin_Headers:Pin_Header_Straight_1x16_Pitch2.54mm" H 5050 5500 50  0001 C CNN
 F 3 "~" H 5050 5500 50  0001 C CNN
 	1    5050 5500
@@
 F 0 "J5" V 7075 5946 50  0000 C CNN
 F 1 "HD44780" V 7166 5946 50  0000 C CNN
-F 2 "lib:PinHeader_1x16_P2.54mm_Vertical" H 6950 6000 50  0001 C CNN
+F 2 "Pin_Headers:Pin_Header_Straight_1x16_Pitch2.54mm" H 6950 6000 50  0001 C CNN
 F 3 "~" H 6950 6000 50  0001 C CNN
 	1    6950 6000
@@
 F 0 "J7" H 2280 5742 50  0000 L CNN
 F 1 "I2C" H 2280 5651 50  0000 L CNN
-F 2 "lib:PinHeader_1x04_P2.54mm_Vertical" H 2200 5750 50  0001 C CNN
+F 2 "Pin_Headers:Pin_Header_Straight_1x04_Pitch2.54mm" H 2200 5750 50  0001 C CNN
 F 3 "~" H 2200 5750 50  0001 C CNN
 	1    2200 5750
@@
 F 0 "U4" H 8850 4100 50  0000 C CNN
 F 1 "STM32F411CEUx" H 8900 4000 50  0000 C CNN
-F 2 "stm32f411ceu6:QFN50P700X700X60-49N-D" H 8250 1950 50  0001 R CNN
+F 2 "lib:stm32f411ceu6" H 8250 1950 50  0001 R CNN
 F 3 "http://www.st.com/st-web-ui/static/active/en/resource/technical/document/datasheet/DM00115249.pdf" H 8850 3450 50  0001 C CNN
 	1    8850 3450
